Commit message: d435 added

File: staubli_tx90_gazebo/urdf/tx90_macro.xacro (robot description, xacro)
@@ -96,4 +96,8 @@
     <turnGravityOff>true</turnGravityOff>
   </gazebo>
+  <gazebo reference="${prefix}tool_link">
+    <material>Gazebo/Grey</material>
+    <turnGravityOff>true</turnGravityOff>
+  </gazebo>
   <!-- ros_control plugin -->
   <gazebo>
@@ -103,4 +107,40 @@
     </plugin>
   </gazebo>
+  <gazebo reference="camera_link">
+    <sensor type="depth" name="camera">
+        <always_on>true</always_on>
+        <update_rate>30.0</update_rate>
+        <camera>
+            <horizontal_fov>${60.0*pi/180.0}</horizontal_fov>
+            <image>
+                <format>R8G8B8</format>
+                <width>640</width>
+                <height>480</height>
+            </image>
+            <clip>
+                <near>0.05</near>
+                <far>8.0</far>
+            </clip>
+        </camera>
+        <plugin name="kinect_camera_controller" filename="libgazebo_ros_openni_kinect.so">
+            <cameraName>camera</cameraName>
+            <alwaysOn>true</alwaysOn>
+            <updateRate>30</updateRate>
+            <imageTopicName>rgb/image_raw</imageTopicName>
+            <depthImageTopicName>depth_registered/image_raw</depthImageTopicName>
+            <pointCloudTopicName>depth_registered/points</pointCloudTopicName>
+            <cameraInfoTopicName>rgb/camera_info</cameraInfoTopicName>
+            <depthImageCameraInfoTopicName>depth_registered/camera_info</depthImageCameraInfoTopicName>
+            <frameName>camera_depth_optical_frame</frameName>
+            <baseline>0.1</baseline>
+            <distortion_k1>0.0</distortion_k1>
+            <distortion_k2>0.0</distortion_k2>
+            <distortion_k3>0.0</distortion_k3>
+            <distortion_t1>0.0</distortion_t1>
+            <distortion_t2>0.0</distortion_t2>
+            <pointCloudCutoff>0.4</pointCloudCutoff>
+        </plugin>
+    </sensor>
+  </gazebo>
   </xacro:macro>
 </robot>

File: staubli_tx90_support/urdf/tx90_macro.xacro (robot description, xacro)
@@ -158,4 +158,30 @@
       </inertial>
     </link>
+  <link name="tool_link">
+    <visual>
+      <origin xyz="0 0 0.001" rpy="0 ${radians(-90.0)} ${radians(180.0)}" />
+      <geometry>
+        <mesh filename="package://gripper_2/meshes/base_link.STL" />
+      </geometry>
+      <material name="">
+        <color
+          rgba="0.75294 0.75294 0.75294 1" />
+      </material>
+    </visual>
+    <collision>
+      <origin xyz="0 0 0.005" rpy="0 ${radians(-90.0)} ${radians(180.0)}" />
+      <geometry>
+        <mesh
+          filename="package://gripper_2/meshes/base_link.STL" />
+      </geometry>
+    </collision>
+    <inertial>
+      <mass value="0.00536" />
+      <origin xyz="0.071574 -1.664E-06 0.013015" rpy="0 0 0" />
+      <inertia ixx="0.000012"  ixy="0.0000000"   ixz="0.0000000"
+                               iyy="0.0013662"   iyz="0.0000000"
+                                                 izz="0.00054605" />
+      </inertial>
+  </link>
     <!-- joints: main serial chain -->
     <joint name="${prefix}joint_1" type="revolute">
@@ -224,11 +250,21 @@
       <child link="${prefix}flange" />
     </joint>
+    <joint name="${prefix}tool_link_fixed" type="fixed">
+        <parent link="${prefix}flange"/>
+        <child link="${prefix}tool_link"/>
+        <origin xyz="0 0 0" rpy="0 ${radians(90.0)} 0"/>
+    </joint>
     <!-- ROS-Industrial 'tool0' frame: all-zeros tool frame -->
-    <link name="${prefix}tool0" />
+    <link name="${prefix}tool_tip_link" />
     <joint name="${prefix}flange-tool0" type="fixed">
-      <origin xyz="0 0 0" rpy="0 ${radians(90.0)} 0" />
-      <parent link="${prefix}flange" />
-      <child link="${prefix}tool0" />
-    </joint>
+      <origin xyz="0 0 0.15" rpy="0 0 0" />
+      <parent link="${prefix}tool_link" />
+      <child link="${prefix}tool_tip_link" />
+    </joint>
+    <!--D435 -->
+  <xacro:include filename="$(find realsense2_description)/urdf/_d435.urdf.xacro" />
+  <xacro:sensor_d435 parent="tool_link" use_nominal_extrinsics="$(arg use_nominal_extrinsics)">
+        <origin xyz="0.17 0 0.05" rpy="0 ${pi} ${pi}"/>
+    </xacro:sensor_d435>
   </xacro:macro>
 </robot>
