Commit message: CFRP sdf visual added

File: staubli_tx90_gazebo/urdf/CFRP.urdf (robot description, URDF)
Before this commit: robot cfrp, 2 links, 1 joints
Links:
- link base_link: geometry collision box size=0.1 0.1 0.0025; visual box size=0.1 0.1 0.0025

File: staubli_tx90_support/urdf/tx90_macro.xacro (robot description, xacro)
@@ -265,5 +265,5 @@
   <xacro:include filename="$(find realsense2_description)/urdf/_d435.urdf.xacro" />
   <xacro:sensor_d435 parent="tool_link" use_nominal_extrinsics="$(arg use_nominal_extrinsics)">
-        <origin xyz="0.17 0 0.05" rpy="0 ${pi} ${pi}"/>
+        <origin xyz="0.13 0 0.057" rpy="0 ${pi} ${pi}"/>
     </xacro:sensor_d435>
   </xacro:macro>

Commit message: cfrp xacro added

File: staubli_tx90_gazebo/urdf/CFRP.urdf (robot description, URDF)
Before this commit: robot cfrp, 2 links, 1 joints
Links:
- removed link base_footprint
- removed link base_link
- added link cfrp_base, mass 1; collision box size=0.1 0.1 0.0025; visual box size=0.1 0.1 0.0025
Joints:
- removed joint base_footprint_fixed

File: staubli_tx90_support/urdf/tx90_macro.xacro (robot description, xacro)
@@ -258,5 +258,5 @@
     <link name="${prefix}tool_tip_link" />
     <joint name="${prefix}flange-tool0" type="fixed">
-      <origin xyz="0 0 0.15" rpy="0 0 0" />
+      <origin xyz="0.15 0 0.15" rpy="0 0 0" />
       <parent link="${prefix}tool_link" />
       <child link="${prefix}tool_tip_link" />
